Commit message: 2

File: src/urdf_example/description/example_gazebo.xacro (robot description, xacro)
@@ -48,7 +48,7 @@
         <child link="camera_link_optical" />
     </joint>
-    <!-- <link name="camera_link_optical"> -->
+    <link name="camera_link_optical"></link>
       <!-- Camera -->
-    <link name="camera_link_optical">
+    <!-- <link name="camera_link_optical">
         <collision>
         <origin xyz="0 0 0" rpy="0 0 0"/>
@@ -69,5 +69,5 @@
         <inertia ixx="1e-6" ixy="0" ixz="0" iyy="1e-6" iyz="0" izz="1e-6" />
         </inertial>
-    </link>
+    </link> -->
     <!-- <xacro:property name="camera_link" value="0.05" /> Size of square 'camera' box -->
     <!-- Add a gazebo tag for the ORIGINAL camera_link (but in the plugin we reference the optical frame so that ROS can orient things correctly) -->
@@ -99,6 +99,6 @@
             <plugin name="camera_controller" filename="libgazebo_ros_camera.so">
                 <frame_name>camera_link_optical</frame_name>
-                <!-- <min_depth>0.1</min_depth>
-                <max_depth>500</max_depth> -->
+                <min_depth>0.1</min_depth>
+                <max_depth>500</max_depth>
                 <!-- <cameraName>rrbot/camera1</cameraName>
                 <imageTopicName>image_raw</imageTopicName>

File: src/urdf_example/description/example_robot.urdf.xacro (robot description, xacro)
@@ -52,5 +52,5 @@
         <axis xyz="1 0 0"/>
         <limit lower="0" upper="2" velocity="100" effort="100"/>
-        <dynamics damping="10.0" friction="10.0"/>
+        <dynamics damping="100.0" friction="10.0"/>
     </joint>
     <!-- slider_link is the box skimming across the top of the base. Its parameters are similar to the base_link, however: -->
@@ -84,5 +84,5 @@
         <axis xyz="0 -1 0"/>
         <limit lower="0" upper="${pi/2}" velocity="100" effort="100"/>
-        <dynamics damping="10.0" friction="10.0"/>
+        <dynamics damping="100.0" friction="10.0"/>
     </joint>
     <!-- arm_link describes the arm -->

Commit message: 3

File: src/urdf_example/description/example_gazebo.xacro (robot description, xacro)
@@ -49,25 +49,4 @@
     </joint>
     <link name="camera_link_optical"></link>
-      <!-- Camera -->
-    <!-- <link name="camera_link_optical">
-        <collision>
-        <origin xyz="0 0 0" rpy="0 0 0"/>
-        <geometry>
-        <box size="${camera_link} ${camera_link} ${camera_link}"/>
-        </geometry>
-        </collision>
-        <visual>
-        <origin xyz="0 0 0" rpy="0 0 0"/>
-        <geometry>
-        <box size="${camera_link} ${camera_link} ${camera_link}"/>
-        </geometry>
-        <material name="red"/>
-        </visual>
-        <inertial>
-        <mass value="1e-5" />
-        <origin xyz="0 0 0" rpy="0 0 0"/>
-        <inertia ixx="1e-6" ixy="0" ixz="0" iyy="1e-6" iyz="0" izz="1e-6" />
-        </inertial>
-    </link> -->
     <!-- <xacro:property name="camera_link" value="0.05" /> Size of square 'camera' box -->
     <!-- Add a gazebo tag for the ORIGINAL camera_link (but in the plugin we reference the optical frame so that ROS can orient things correctly) -->
@@ -85,5 +64,5 @@
                     <width>640</width>
                     <height>480</height>
-                    <format>R8B8G8</format>
+                    <format>R8G8B8</format>
                 </image>
                 <clip>
@@ -101,14 +80,4 @@
                 <min_depth>0.1</min_depth>
                 <max_depth>500</max_depth>
-                <!-- <cameraName>rrbot/camera1</cameraName>
-                <imageTopicName>image_raw</imageTopicName>
-                <cameraInfoTopicName>camera_info</cameraInfoTopicName>
-                <frameName>camera_link</frameName>
-                <hackBaseline>0.07</hackBaseline>
-                <distortionK1>0.0</distortionK1>
-                <distortionK2>0.0</distortionK2>
-                <distortionK3>0.0</distortionK3>
-                <distortionT1>0.0</distortionT1>
-                <distortionT2>0.0</distortionT2> -->
             </plugin>
         </sensor>

File: src/urdf_example/description/example_robot.urdf.xacro (robot description, xacro)
@@ -52,5 +52,5 @@
         <axis xyz="1 0 0"/>
         <limit lower="0" upper="2" velocity="100" effort="100"/>
-        <dynamics damping="100.0" friction="10.0"/>
+        <!-- <dynamics damping="10.0" friction="10.0"/> -->
     </joint>
     <!-- slider_link is the box skimming across the top of the base. Its parameters are similar to the base_link, however: -->
@@ -84,5 +84,5 @@
         <axis xyz="0 -1 0"/>
         <limit lower="0" upper="${pi/2}" velocity="100" effort="100"/>
-        <dynamics damping="100.0" friction="10.0"/>
+        <!-- <dynamics damping="10.0" friction="10.0"/> -->
     </joint>
     <!-- arm_link describes the arm -->

Commit message: 5

File: src/urdf_example/description/example_gazebo.xacro (robot description, xacro)
@@ -56,5 +56,5 @@
             try swapping "depth" to "camera"-->
     <gazebo reference="camera_link">
-        <sensor type="camera" name="my_camera">
+        <sensor type="depth" name="my_camera">
             <update_rate>20</update_rate>
             <visualize>true</visualize>

File: src/urdf_example/description/example_robot.urdf.xacro (robot description, xacro)
@@ -52,5 +52,5 @@
         <axis xyz="1 0 0"/>
         <limit lower="0" upper="2" velocity="100" effort="100"/>
-        <!-- <dynamics damping="10.0" friction="10.0"/> -->
+        <dynamics damping="10.0" friction="10.0"/>
     </joint>
     <!-- slider_link is the box skimming across the top of the base. Its parameters are similar to the base_link, however: -->
@@ -84,5 +84,5 @@
         <axis xyz="0 -1 0"/>
         <limit lower="0" upper="${pi/2}" velocity="100" effort="100"/>
-        <!-- <dynamics damping="10.0" friction="10.0"/> -->
+        <dynamics damping="10.0" friction="10.0"/>
     </joint>
     <!-- arm_link describes the arm -->
